Commit message: 7th commit

File: src/4-wheel-differential-car-ros/carmodel_description/urdf/robot.urdf (robot description, URDF)
Before this commit: robot differential_drive_robot, 6 links, 5 joints
Joints:
- joint wheel1_joint: type continious -> continuous
- joint wheel2_joint: type continious -> continuous
- joint wheel3_joint: origin xyz=${body_link_x_dim/2+1.2*wheel_link_radius} ${-body_link_y_dim/2-wheel_link_length/2} $ {wheel_link_z_location} rpy=0 0 0 -> xyz=${body_link_x_dim/2+1.2*wheel_link_radius} ${-body_link_y_dim/2-wheel_link_length/2} ${wheel_link_z_location} rpy=0 0 0; type continious -> continuous
- joint wheel4_joint: type continious -> continuous
