Commit message: 8th commit

File: src/4-wheel-differential-car-ros/carmodel_description/urdf/carmodel2.urdf (robot description, URDF)
Before this commit: robot carmodel, 7 links, 6 joints
Links:
- link base_link: mass 65.8282 -> 10; geometry collision box size=0.8 0.3 0.1; visual box size=0.8 0.3 0.1
- link wheel_1: mass 1.0252 -> 2.5; geometry collision cylinder length=0.2 radius=0.1; visual cylinder length=0.2 radius=0.1
- link wheel_2: mass 1.252 -> 2.5; geometry collision cylinder length=0.2 radius=0.1; visual cylinder length=0.2 radius=0.1
- link wheel_3: mass 1.252 -> 2.5; geometry collision cylinder length=0.2 radius=0.1; visual cylinder length=0.2 radius=0.1
- link wheel_4: mass 1.252 -> 2.5; geometry collision cylinder length=0.2 radius=0.1; visual cylinder length=0.2 radius=0.1
Joints:
- removed joint joint_base_wheel1
- removed joint joint_base_wheel2
- removed joint joint_base_wheel3
- removed joint joint_base_wheel4
- added joint body_to_left_front: type continuous, parent base_link, child wheel_1, origin xyz=0.38 0.15 0 rpy=0 0 0, axis 0 1 0
- added joint body_to_left_rear: type continuous, parent base_link, child wheel_3, origin xyz=-0.38 0.15 0 rpy=0 0 0, axis 0 1 0
- added joint body_to_right_front: type continuous, parent base_link, child wheel_2, origin xyz=0.38 -0.15 0 rpy=0 0 0, axis 0 1 0
- added joint body_to_right_rear: type continuous, parent base_link, child wheel_4, origin xyz=-0.38 -0.15 0 rpy=0 0 0, axis 0 1 0

Commit message: 9th commit

File: src/4-wheel-differential-car-ros/carmodel_description/urdf/carmodel2.urdf (robot description, URDF)
Before this commit: robot carmodel, 7 links, 6 joints
Joints:
- removed joint body_to_left_front
- removed joint body_to_left_rear
- removed joint body_to_right_front
- removed joint body_to_right_rear
- added joint joint_base_wheel1: type continuous, parent base_link, child wheel_1, origin xyz=0.38 -0.15 0 rpy=0 0 0, axis 0 1 0
- added joint joint_base_wheel2: type continuous, parent base_link, child wheel_2, origin xyz=-0.38 -0.15 0 rpy=0 0 0, axis 0 1 0
- added joint joint_base_wheel3: type continuous, parent base_link, child wheel_3, origin xyz=0.38 0.15 0 rpy=0 0 0, axis 0 1 0
- added joint joint_base_wheel4: type continuous, parent base_link, child wheel_4, origin xyz=-0.38 0.15 0 rpy=0 0 0, axis 0 1 0

Commit message: 11th fix

File: src/4-wheel-differential-car-ros/carmodel_description/urdf/carmodel2.urdf (robot description, URDF)
Before this commit: robot carmodel, 7 links, 6 joints
Links:
- link wheel_1: geometry collision cylinder length=0.06 radius=0.1; visual cylinder length=0.06 radius=0.1
- link wheel_2: geometry collision cylinder length=0.06 radius=0.1; visual cylinder length=0.06 radius=0.1
- link wheel_3: geometry collision cylinder length=0.06 radius=0.1; visual cylinder length=0.06 radius=0.1
- link wheel_4: geometry collision cylinder length=0.06 radius=0.1; visual cylinder length=0.06 radius=0.1

Commit message: fix all

File: src/4-wheel-differential-car-ros/carmodel_description/urdf/carmodel2.urdf (robot description, URDF)
Before this commit: robot carmodel, 7 links, 6 joints
Links:
- added link sensor_link, mass 3; collision cylinder length=0.1 radius=0.05; visual cylinder length=0.1 radius=0.05
Joints:
- added joint sensor_joint: type fixed, parent base_link, child sensor_link, origin xyz=0.15 0 0.05 rpy=0 0 0

File: src/4-wheel-differential-car-ros/carmodel_description/urdf/carmodel2.urdf.xacro (robot description, xacro)
@@ -4,4 +4,7 @@
   <xacro:property name="wheel_radius" value="0.03018"/>
   <xacro:property name="width" value="0.13189"/>
+    <gazebo reference="sensor_link">
+      <material>Gazebo/Red</material>
+    </gazebo>
     <gazebo reference="base_link">
       <material>Gazebo/Orange</material>
@@ -114,4 +117,39 @@
     </sensor>
   </gazebo>
+  <gazebo reference="sensor_link">
+    <sensor type="ray" name="head_hokuyo_sensor">
+    <pose>0 0 0 0 0 0</pose>
+    <visualize>true</visualize>
+    <update_rate>20</update_rate>
+    <ray>
+        <scan>
+        <horizontal>
+            <samples>720</samples>
+            <resolution>1</resolution>
+            <min_angle>-1.04719755</min_angle>
+            <max_angle>1.04719755</max_angle>
+        </horizontal>
+        </scan>
+        <range>
+        <min>0.10</min>
+        <max>2.0</max>
+        <resolution>0.01</resolution>
+        </range>
+        <noise>
+        <type>gaussian</type>
+        <!-- Noise parameters based on published spec for Hokuyo laser
+            achieving "+-30mm" accuracy at range < 10m.  A mean of 0.0m and
+            stddev of 0.01m will put 99.7% of samples within 0.03m of the true
+            reading. -->
+        <mean>0.0</mean>
+        <stddev>0.01</stddev>
+        </noise>
+    </ray>
+    <plugin name="gazebo_ros_head_hokuyo_controller" filename="libgazebo_ros_laser.so">
+        <topicName>/m2wr/laser/scan</topicName>
+        <frameName>sensor_link</frameName>
+    </plugin>
+    </sensor>
+  </gazebo>
   <carmodel/>
 </robot>
