Commit message: update roller and wheel

File: src/4-wheel-differential-car-ros/carmodel_description/urdf/rollers.xacro (robot description, xacro)
@@ -15,10 +15,10 @@
           <origin xyz="0 0 0" rpy="0 0 0" />
           <geometry>
-            <mesh filename="package://fuji_mecanum/mesh/visual/roller.dae" scale="1 1 1" />
+            <mesh filename="package://carmodel_description/mesh/visual/roller.dae" scale="1 1 1" />
           </geometry>
         </visual>
         <collision>
           <geometry>
-            <mesh filename="package://fuji_mecanum/mesh/collision/roller.stl" scale="1 1 1" />
+            <mesh filename="package://carmodel_description/mesh/collision/roller.stl" scale="1 1 1" />
           </geometry>
         </collision>

File: src/4-wheel-differential-car-ros/carmodel_description/urdf/wheel.xacro (robot description, xacro)
@@ -6,10 +6,10 @@
         <origin xyz="0 0 0" rpy="0 0 0" />
         <geometry>
-          <mesh filename="package://fuji_mecanum/mesh/visual/wheel.dae" scale="${side} 1 1" />
+          <mesh filename="package://carmodel_description/mesh/visual/wheel.dae" scale="${side} 1 1" />
         </geometry>
       </visual>
       <collision>
         <geometry>
-          <mesh filename="package://fuji_mecanum/mesh/collision/wheel.stl" scale="${side} 1 1" />
+          <mesh filename="package://carmodel_description/mesh/collision/wheel.stl" scale="${side} 1 1" />
         </geometry>
       </collision>
