Commit message: modifile stl and change urdf

File: src/4-wheel-differential-car-ros/carmodel_description/urdf/bot_description.xacro (robot description, xacro)
@@ -6,4 +6,5 @@
 <xacro:include filename="$(find carmodel_description)/urdf/gazebo.xacro" />
 <xacro:include filename="$(find carmodel_description)/urdf/link_joint.xacro" />
+<xacro:include filename="$(find carmodel_description)/urdf/mecanum_wheel_macro.xacro" />
   <link name="link_chassis">
     <!-- pose and inertial -->
@@ -54,17 +55,28 @@
   <!-- Create sensor joint -->
   <xacro:sensor_joint />
-  <!-- Create wheel right -->
-  <xacro:link_wheel name="link_right_wheel" />
+  <xacro:mecanum_wheel name="front_right" side="1"  interface="hardware_interface/EffortJointInterface"/>
+  <xacro:mecanum_wheel name="front_left"  side="-1" interface="hardware_interface/EffortJointInterface"/>
+  <xacro:mecanum_wheel name="rear_right"  side="-1" interface="hardware_interface/EffortJointInterface"/>
+  <xacro:mecanum_wheel name="rear_left"   side="1"  interface="hardware_interface/EffortJointInterface"/>
   <!-- Create joint right -->
+  <xacro:joint_wheel name="rear_right_wheel_joint" param_xyz="-0.15 0.15 0" child="rear_right_wheel_link"  />
+  <!-- Create joint left -->
+  <xacro:joint_wheel name="rear_left_wheel_joint" param_xyz="-0.15 -0.15 0" child="rear_left_wheel_link"  />
+  <xacro:joint_wheel name="front_left_wheel_joint" param_xyz="0.13 -0.15 0" child="front_left_wheel_link"  />
+  <xacro:joint_wheel name="front_right_wheel_joint" param_xyz="0.13 0.15 0" child="front_right_wheel_link"  />
+  <!-- Create wheel right
+  <xacro:wheel_link name="link_right_wheel" />
+   Create joint right
   <xacro:joint_wheel name="joint_right_wheel" param_xyz="-0.15 0.15 0" child="link_right_wheel"  />
-  <!-- Create wheel left -->
-  <xacro:link_wheel name="link_left_wheel" />
-  <!-- Create joint left -->
+  Create wheel left
+  <xacro:wheel_link name="link_left_wheel" />
+   Create joint left
   <xacro:joint_wheel name="joint_left_wheel" param_xyz="-0.15 -0.15 0" child="link_left_wheel"  />
-  <!-- front left-->
-  <xacro:link_wheel name="link_front_left_wheel" />
+   front left
+  <xacro:wheel_link name="link_front_left_wheel" />
   <xacro:joint_wheel name="joint_front_left_wheel" param_xyz="0.13 -0.15 0" child="link_front_left_wheel"  />
-  <!--front right-->
-  <xacro:link_wheel name="link_front_right_wheel" />
-  <xacro:joint_wheel name="joint_front_right_wheel" param_xyz="0.13 0.15 0" child="link_front_right_wheel"  />
+  front right
+  <xacro:wheel_link
+   name="link_front_right_wheel" />
+  <xacro:joint_wheel name="joint_front_right_wheel" param_xyz="0.13 0.15 0" child="link_front_right_wheel"  /> -->
 </robot>

File: src/4-wheel-differential-car-ros/carmodel_description/urdf/gazebo.xacro (robot description, xacro)
@@ -4,8 +4,8 @@
         <material>Gazebo/Orange</material>
     </gazebo>
-    <gazebo reference="link_left_wheel">
+    <gazebo reference="rear_left_wheel_link">
         <material>Gazebo/Blue</material>
     </gazebo>
-    <gazebo reference="link_right_wheel">
+    <gazebo reference="rear_right_wheel_link">
         <material>Gazebo/Blue</material>
     </gazebo>
@@ -14,8 +14,8 @@
     </gazebo>
     <!--test them banh-->
-    <gazebo reference="link_front_right_wheel">
+    <gazebo reference="front_right_wheel_link">
         <material>Gazebo/Blue</material>
     </gazebo>
-    <gazebo reference="link_front_left_wheel">
+    <gazebo reference="front_left_wheel_link">
         <material>Gazebo/Blue</material>
     </gazebo>
@@ -25,6 +25,6 @@
         <alwaysOn>true</alwaysOn>
         <updateRate>20</updateRate>
-        <leftJoint>joint_left_wheel</leftJoint>
-        <rightJoint>joint_right_wheel</rightJoint>
+        <leftJoint>rear_left_wheel_joint</leftJoint>
+        <rightJoint>rear_right_wheel_joint</rightJoint>
         <wheelSeparation>0.6</wheelSeparation>
         <wheelDiameter>0.2</wheelDiameter>
@@ -97,4 +97,5 @@
         </plugin>
     </gazebo> -->
+    <!-- lay tu mobile mecanum-->
         <gazebo>
         <plugin name="object_controller" filename="libgazebo_ros_planar_move.so">
@@ -104,8 +105,8 @@
             <robotBaseFrame>base_footprint</robotBaseFrame>
             <!-- Wheel Information -->
-            <left_joint>joint_left_wheel</left_joint>
-            <right_joint>joint_right_wheel</right_joint>
-            <left_joint>joint_front_left_wheel</left_joint>
-            <right_joint>joint_front_right_wheel</right_joint>
+            <left_joint>rear_left_wheel_joint</left_joint>
+            <right_joint>rear_right_wheel_joint</right_joint>
+            <left_joint>front_left_wheel_joint</left_joint>
+            <right_joint>front_right_wheel_joint</right_joint>
             <wheel_separation>0.35</wheel_separation>
             <wheel_diameter>0.1</wheel_diameter>

File: src/4-wheel-differential-car-ros/carmodel_description/urdf/link_joint.xacro (robot description, xacro)
@@ -1,26 +1,4 @@
 <?xml version="1.0" ?>
 <robot name="m2wr" xmlns:xacro="https://www.ros.org/wiki/xacro" >   <!-- this second parameter is importent to make this file a valid xacro file -->
-    <xacro:macro name="link_wheel" params="name">
-    <!-- phan thiet ke banh xe-->
-    <link name="${name}">
-            <inertial>
-            <mass value="0.2"/>
-            <origin rpy="0 1.5707 1.5707" xyz="0 0 0"/>
-            <inertia ixx="0.00052666666" ixy="0" ixz="0" iyy="0.052666666" iyz="0" izz="0.001"/>
-            </inertial>
-            <collision name="${name}_collision">
-            <origin rpy="0 1.5707 1.5707" xyz="0 0 0" />
-            <geometry>
-                <cylinder length="0.04" radius="0.1"/>
-            </geometry>
-            </collision>
-            <visual name="${name}_visual">
-            <origin rpy="0 1.5707 1.5707" xyz="0 0 0"/>
-            <geometry>
-                <cylinder length="0.04" radius="0.1"/>
-            </geometry>
-            </visual>
-        </link>
-    </xacro:macro>
     <xacro:macro name="joint_wheel" params="name param_xyz child">
         <joint name="${name}" type="continuous">

Commit message: hoan thien model

File: src/4-wheel-differential-car-ros/carmodel_description/urdf/bot_description.xacro (robot description, xacro)
@@ -27,27 +27,4 @@
       <material name="blue"/>
     </visual>
-    <!-- caster front -->
-    <collision name = "caster_front_collision">
-      <origin rpy=" 0 0 0" xyz="0.35 0 -0.05"/>
-      <geometry>
-        <sphere radius="0.05"/>
-      </geometry>
-      <surface>
-        <friction>
-          <ode>
-            <mu>0</mu>
-            <mu2>0</mu2>
-            <slip1>1.0</slip1>
-            <slip2>1.0</slip2>
-          </ode>
-        </friction>
-      </surface>
-    </collision>
-    <visual name="caster_front_visual">
-      <origin rpy=" 0 0 0" xyz="0.2 0 -0.05"/>
-      <geometry>
-        <sphere radius="0.05"/>
-      </geometry>
-    </visual>
   </link>
   <!-- Create sensor link  -->
@@ -59,10 +36,28 @@
   <xacro:mecanum_wheel name="rear_right"  side="-1" interface="hardware_interface/EffortJointInterface"/>
   <xacro:mecanum_wheel name="rear_left"   side="1"  interface="hardware_interface/EffortJointInterface"/>
-  <!-- Create joint right -->
-  <xacro:joint_wheel name="rear_right_wheel_joint" param_xyz="-0.15 0.15 0" child="rear_right_wheel_link"  />
-  <!-- Create joint left -->
-  <xacro:joint_wheel name="rear_left_wheel_joint" param_xyz="-0.15 -0.15 0" child="rear_left_wheel_link"  />
-  <xacro:joint_wheel name="front_left_wheel_joint" param_xyz="0.13 -0.15 0" child="front_left_wheel_link"  />
-  <xacro:joint_wheel name="front_right_wheel_joint" param_xyz="0.13 0.15 0" child="front_right_wheel_link"  />
+  <joint name="front_right_wheel_joint" type="continuous">
+    <origin xyz="0.15 -0.19 0" rpy="0 0 ${pi/2}" />
+    <axis xyz="1 0 0" />
+    <parent link="link_chassis" />
+    <child link="front_right_wheel_link" />
+  </joint>
+  <joint name="front_left_wheel_joint" type="continuous">
+    <origin xyz="0.15 0.19 0" rpy="0 0 ${pi/2}" />
+    <axis xyz="1 0 0" />
+    <parent link="link_chassis" />
+    <child link="front_left_wheel_link" />
+  </joint>
+  <joint name="rear_right_wheel_joint" type="continuous">
+    <origin xyz="-0.15 -0.19 0" rpy="0 0 ${pi/2}" />
+    <axis xyz="1 0 0" />
+    <parent link="link_chassis" />
+    <child link="rear_right_wheel_link" />
+  </joint>
+  <joint name="rear_left_wheel_joint" type="continuous">
+    <origin xyz="-0.15 0.19 0" rpy="0 0 ${pi/2}" />
+    <axis xyz="1 0 0" />
+    <parent link="link_chassis" />
+    <child link="rear_left_wheel_link" />
+  </joint>
   <!-- Create wheel right
   <xacro:wheel_link name="link_right_wheel" />

File: src/4-wheel-differential-car-ros/carmodel_description/urdf/link_joint.xacro (robot description, xacro)
@@ -1,14 +1,15 @@
 <?xml version="1.0" ?>
 <robot name="m2wr" xmlns:xacro="https://www.ros.org/wiki/xacro" >   <!-- this second parameter is importent to make this file a valid xacro file -->
-    <xacro:macro name="joint_wheel" params="name param_xyz child">
+<!-- old joint-link wheel -->
+ <!--   <xacro:macro name="joint_wheel" params="name param_xyz child">
         <joint name="${name}" type="continuous">
-            <origin rpy="0 0 0" xyz="${param_xyz}"/>        <!-- this gives orientation -->
+            <origin rpy="0 0 0" xyz="${param_xyz}"/>
             <child link="${child}" />
             <parent link="link_chassis"/>
-            <axis rpy="0 0 0" xyz="0 1 0"/>    <!-- this says rotate about y axis -->
+            <axis rpy="0 0 0" xyz="0 1 0"/>
             <limit effort="10000" velocity="1000"/>
             <joint_properties damping="1.0" friction="1.0" />
         </joint>
-    </xacro:macro>
+    </xacro:macro> -->
     <xacro:macro name="sensor_link">
         <link name = "sensor_link">

File: src/4-wheel-differential-car-ros/carmodel_description/urdf/mecanum_wheel_macro.xacro (robot description, xacro)
@@ -2,5 +2,5 @@
 <robot name="mecanum_wheel" xmlns:xacro="http://ros.org/wiki/xacro">
   <xacro:include filename="$(find carmodel_description)/urdf/wheel.xacro" />
-  <xacro:include filename="$(find carmodel-description)/urdf/rollers.xacro"  />
+  <xacro:include filename="$(find carmodel_description)/urdf/rollers.xacro"  />
   <xacro:macro name="mecanum_wheel" params="name side interface">
     <xacro:wheel_link name="${name}" side="${side}" />

File: src/4-wheel-differential-car-ros/carmodel_description/urdf/rollers.xacro (robot description, xacro)
@@ -15,10 +15,10 @@
           <origin xyz="0 0 0" rpy="0 0 0" />
           <geometry>
-            <mesh filename="package://carmodel_description/mesh/visual/roller.dae" scale="1 1 1" />
+            <mesh filename="package://carmodel_description/meshes/visual/roller.dae" scale="1 1 1" />
           </geometry>
         </visual>
         <collision>
           <geometry>
-            <mesh filename="package://carmodel_description/mesh/collision/roller.stl" scale="1 1 1" />
+            <mesh filename="package://carmodel_description/meshes/collision/roller.stl" scale="1 1 1" />
           </geometry>
         </collision>

File: src/4-wheel-differential-car-ros/carmodel_description/urdf/wheel.xacro (robot description, xacro)
@@ -6,10 +6,10 @@
         <origin xyz="0 0 0" rpy="0 0 0" />
         <geometry>
-          <mesh filename="package://carmodel_description/mesh/visual/wheel.dae" scale="${side} 1 1" />
+          <mesh filename="package://carmodel_description/meshes/visual/wheel.dae" scale="${side} 1 1" />
         </geometry>
       </visual>
       <collision>
         <geometry>
-          <mesh filename="package://carmodel_description/mesh/collision/wheel.stl" scale="${side} 1 1" />
+          <mesh filename="package://carmodel_description/meshes/collision/wheel.stl" scale="${side} 1 1" />
         </geometry>
       </collision>

Commit message: fix camera and plugin

File: src/4-wheel-differential-car-ros/carmodel_description/urdf/bot_description.xacro (robot description, xacro)
@@ -7,5 +7,10 @@
 <xacro:include filename="$(find carmodel_description)/urdf/link_joint.xacro" />
 <xacro:include filename="$(find carmodel_description)/urdf/mecanum_wheel_macro.xacro" />
-  <link name="link_chassis">
+<xacro:include filename="$(find carmodel_description)/urdf/_t265.urdf.xacro"/>
+  <xacro:sensor_t265  parent="base_link" name="T265_camera" topics_ns="T265_camera"
+                      odom_xyz="0.0 0.0 0.25" odom_rpy="0.0 0.0 0.0">
+    <origin xyz="0.0 0.0 0.25" rpy="0.0 0.0 0.0"/>
+  </xacro:sensor_t265>
+  <link name="base_link">
     <!-- pose and inertial -->
     <pose>0 0 0.1 0 0 0</pose>
@@ -39,5 +44,5 @@
     <origin xyz="0.15 -0.19 0" rpy="0 0 ${pi/2}" />
     <axis xyz="1 0 0" />
-    <parent link="link_chassis" />
+    <parent link="base_link" />
     <child link="front_right_wheel_link" />
   </joint>
@@ -45,5 +50,5 @@
     <origin xyz="0.15 0.19 0" rpy="0 0 ${pi/2}" />
     <axis xyz="1 0 0" />
-    <parent link="link_chassis" />
+    <parent link="base_link" />
     <child link="front_left_wheel_link" />
   </joint>
@@ -51,5 +56,5 @@
     <origin xyz="-0.15 -0.19 0" rpy="0 0 ${pi/2}" />
     <axis xyz="1 0 0" />
-    <parent link="link_chassis" />
+    <parent link="base_link" />
     <child link="rear_right_wheel_link" />
   </joint>
@@ -57,5 +62,5 @@
     <origin xyz="-0.15 0.19 0" rpy="0 0 ${pi/2}" />
     <axis xyz="1 0 0" />
-    <parent link="link_chassis" />
+    <parent link="base_link" />
     <child link="rear_left_wheel_link" />
   </joint>

File: src/4-wheel-differential-car-ros/carmodel_description/urdf/gazebo.xacro (robot description, xacro)
@@ -1,5 +1,5 @@
 <?xml version="1.0" ?>
 <robot name="m2wr" xmlns:xacro="https://www.ros.org/wiki/xacro" >   <!-- this second parameter is importent to make this file a valid xacro file -->
-    <gazebo reference="link_chassis">
+    <gazebo reference="base_link">
         <material>Gazebo/Orange</material>
     </gazebo>
@@ -33,5 +33,5 @@
         <odometryTopic>odom</odometryTopic>
         <odometryFrame>odom</odometryFrame>
-        <robotBaseFrame>link_chassis</robotBaseFrame>
+        <robotBaseFrame>base_link</robotBaseFrame>
         </plugin>
     </gazebo>

File: src/4-wheel-differential-car-ros/carmodel_description/urdf/link_joint.xacro (robot description, xacro)
@@ -6,5 +6,5 @@
             <origin rpy="0 0 0" xyz="${param_xyz}"/>
             <child link="${child}" />
-            <parent link="link_chassis"/>
+            <parent link="base_link"/>
             <axis rpy="0 0 0" xyz="0 1 0"/>
             <limit effort="10000" velocity="1000"/>
@@ -37,5 +37,5 @@
         <joint name="sensor_joint" type="fixed">
             <origin xyz="0.15 0 0.05" rpy="0 0 0"/>
-            <parent link="link_chassis"/>
+            <parent link="base_link"/>
             <child link="sensor_link"/>
         </joint>

Commit message: fix parameter cam

File: src/4-wheel-differential-car-ros/carmodel_description/urdf/bot_description.xacro (robot description, xacro)
@@ -9,6 +9,6 @@
 <xacro:include filename="$(find carmodel_description)/urdf/_t265.urdf.xacro"/>
   <xacro:sensor_t265  parent="base_link" name="T265_camera" topics_ns="T265_camera"
-                      odom_xyz="0.0 0.0 0.25" odom_rpy="0.0 0.0 0.0">
-    <origin xyz="0.0 0.0 0.25" rpy="0.0 0.0 0.0"/>
+                      odom_xyz="0.0 0 0.25" odom_rpy="0.0 0.0 0.0">
+    <origin xyz="0.18 0.0 0.116" rpy="0.0 0.0 0.0"/>
   </xacro:sensor_t265>
   <link name="base_link">

File: src/4-wheel-differential-car-ros/carmodel_description/urdf/link_joint.xacro (robot description, xacro)
@@ -24,5 +24,5 @@
                 <cylinder radius="0.05" length="0.1" />
                 </geometry>
-                <material name="Cyan"/>
+                <material name="Gazebo/Cyan"/>
             </visual>
             <collision>

Commit message: update source code

File: src/4-wheel-differential-car-ros/carmodel_description/urdf/bot_description.xacro (robot description, xacro)
@@ -15,5 +15,5 @@
   <link name="base_link">
     <!-- pose and inertial -->
-    <pose>0 0 0.1 0 0 0</pose>
+    <pose>0 0 0 0 0 0</pose>
     <inertial>
       <mass value="5"/>

File: src/4-wheel-differential-car-ros/carmodel_description/urdf/example.urdf.xacro (robot description, xacro)
@@ -11,13 +11,13 @@
    <parent link="base_footprint" />
     <child link="base_link" />
-    <origin xyz="0 0 0.05" rpy="0 0 0" />
+    <origin xyz="0 0 0" rpy="0 0 0" />
   </joint>
   <xacro:include filename="$(find carmodel_description)/urdf/VLP-16.urdf.xacro"/>
   <xacro:VLP-16 parent="base_link" name="velodyne" topic="/velodyne_points" organize_cloud="${organize_cloud}" hz="10" samples="440" gpu="${gpu}">
-    <origin xyz="0 0 0.4" rpy="0 0 0" />
+    <origin xyz="0 0 0" rpy="0 0 0" />
   </xacro:VLP-16>
   <xacro:include filename="$(find carmodel_description)/urdf/HDL-32E.urdf.xacro"/>
   <xacro:HDL-32E parent="base_link" name="velodyne2" topic="/velodyne_points2" organize_cloud="${organize_cloud}" hz="10" samples="220" gpu="${gpu}">
-    <origin xyz="0 0 0.6" rpy="0 0 0" />
+    <origin xyz="0 0 0" rpy="0 0 0" />
   </xacro:HDL-32E>
 </robot>
